Commit message: finish_for_meeting

File: urdf/robot_body.urdf (robot description, URDF)
Before this commit: robot arm_robot, 9 links, 8 joints
Joints:
- joint arm2_joint: limit lower=-1.5 upper=1.5 effort=30 velocity=1.5 -> lower=-2.0 upper=2.0 effort=30 velocity=1.5
- joint arm3_joint: limit lower=-1.7 upper=1.7 effort=30 velocity=1.5 -> lower=-1.7 upper=2.26 effort=30 velocity=1.5
